Commit message: add damping and frinction

File: rcg/urdf/wheel.urdf.xacro (robot description, xacro)
@@ -93,5 +93,5 @@
       <origin xyz="${xyz}" rpy="${rpy}" />
       <axis xyz="0 0 1" />
-      <!-- <dynamics damping="0.1" friction="0.05"/> -->
+      <dynamics damping="0.1" friction="0.1"/>
     </joint>
     <!-- Link -->
